File: hardware/esp32ValveControl/esp32ValveControl.kicad_pcb (KiCad board)
At the start: 2 copper layers, 50 x 86.5 mm, 61 parts, among them Q1 BSS138, Q2 BSS138, Q5 BSS138, Q7 BSS138, SW2 Reset, U1 ESP32-WROOM, U2 AQY212, U3 AQY212, U4 MC34063, U5 MOCD207M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

Commit message: schem_/pcb update
Parts:
- removed D1, D2, D3: LED, LEDs:LED-0603
- added C1: 100n, Capacitors_SMD:C_0603, F.Cu at (71.9, 79.7)
- added P1: CONN_01X05, Pin_Headers:Pin_Header_Straight_1x05_Pitch2.54mm, F.Cu at (96.0, 81.0)
- added R1: 10k, Resistors_SMD:R_0603, F.Cu at (74.5, 91.1)
- added R2: 10k, Resistors_SMD:R_0603, F.Cu at (82.1, 91.1)
- added R23: 100, Resistors_SMD:R_0603, F.Cu at (65.6, 58.1)
- added R6: 10k, Resistors_SMD:R_0603, F.Cu at (89.7, 91.1)
- added R7: 10k, Resistors_SMD:R_0603, F.Cu at (97.3, 91.1)
- added SW1: Boot, switches:SMD_Switch_6.5x6, F.Cu at (57.9, 55.6)
- added U8: MOCD207M, Housings_SOIC:SOIC-8_3.9x4.9mm_Pitch1.27mm, F.Cu at (82.1, 53.0)
- R18, R19, R22, R3, R4, R5: value 470 -> 10k
- R20, R21: value 470 -> tbd
- R8, R9: value 33 -> 10k
- U2, U3, U6, U7: footprint TO_SOT_Packages_SMD:SOT-428 -> Housings_DIP:DIP-4_W7.62mm_SMDSocket_SmallPads
- moved R15 42.2 mm to (52.9, 49.2), turned to 90 degrees
- moved D6 40.4 mm to (56.7, 49.2), turned to 0 degrees
- moved R8 37.3 mm to (87.2, 50.5), turned to 90 degrees
- moved R16 36.9 mm to (56.7, 51.8), turned to 180 degrees
- moved R22 36.0 mm to (73.2, 79.7), turned to 270 degrees
- moved R9 31.5 mm to (77.0, 55.6), turned to 180 degrees
- moved U7 24.0 mm to (96.0, 98.7), turned to 270 degrees
- moved U2 24.0 mm to (73.2, 98.7), turned to 270 degrees
- moved R5 23.5 mm to (80.8, 47.9), turned to 0 degrees
- moved D12 22.9 mm to (73.9, 84.1)
- moved D15 22.9 mm to (96.2, 84.0)
- moved Q1 22.9 mm to (74.0, 86.6)
- moved Q7 22.9 mm to (96.1, 86.4)
- moved R33 22.9 mm to (76.8, 86.5)
- moved R36 22.9 mm to (98.8, 86.5)
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Connections:
- D10 pad 1: /OUT3 -> /OUT2
- D11 pad 1: /OUT4 -> /OUT1
- D8 pad 1: /OUT1 -> /OUT4
- D9 pad 1: /OUT2 -> /OUT3
- R18 pad 1: /nReset -> /OPTO4
- R18 pad 2: Net-(R18-Pad2) -> +3V3
- R19 pad 1: /PE1 -> +3V3
- R20 pad 1: /PE0 -> /IN3
- R21 pad 1: /PD6 -> /IN4
- R22 pad 1: /PD7 -> /nBoot
- R22 pad 2: Net-(R22-Pad2) -> +3V3
- R3 pad 1: Net-(D1-Pad2) -> Net-(R3-Pad1)
- R3 pad 2: +3V3 -> /IN1
- R4 pad 1: Net-(D2-Pad2) -> Net-(R4-Pad1)
- R4 pad 2: +3V3 -> /IN2
- R5 pad 2: +3V3 -> /IN3
- R8 pad 2: /CH3 -> /IN4
- R9 pad 1: Net-(R9-Pad1) -> /OPTO3
- R9 pad 2: /CH4 -> +3V3
- U1 pad 1: Net-(U1-Pad1) -> GND
- U1 pad 15: Net-(U1-Pad15) -> GND
- U1 pad 2: Net-(U1-Pad2) -> +3V3
- U1 pad 25: Net-(U1-Pad25) -> /nBoot
- U1 pad 27: Net-(U1-Pad27) -> /CH1
- U1 pad 28: Net-(U1-Pad28) -> /CH2
- U1 pad 29: Net-(U1-Pad29) -> /CH3
- U1 pad 3: Net-(U1-Pad3) -> Net-(R19-Pad2)
- U1 pad 30: Net-(U1-Pad30) -> /CH4
- U1 pad 38: Net-(U1-Pad38) -> GND
- U1 pad 39: Net-(U1-Pad39) -> GND
- U5 pad 1: /IN1 -> Net-(R3-Pad1)
- U5 pad 2: GND -> VCOM
- U5 pad 3: /IN2 -> Net-(R4-Pad1)
- U5 pad 4: GND -> VCOM
- X1 pad 10: +24V -> /Vin
- X1 pad 11: Net-(R31-Pad2) -> GND
- X1 pad 12: Net-(R32-Pad2) -> +24V
- X1 pad 13: Net-(R18-Pad2) -> GND
- X1 pad 14: Net-(R19-Pad2) -> Net-(R31-Pad2)
- X1 pad 15: Net-(R20-Pad2) -> Net-(R32-Pad2)
- X1 pad 16: Net-(R21-Pad2) -> Net-(R20-Pad2)
- X1 pad 17: Net-(R22-Pad2) -> Net-(R21-Pad2)
- X1 pad 18: GND -> VCOM
- X1 pad 2: /Vin -> /OUT1
- X1 pad 3: /Vin -> GND
- X1 pad 4: /Vin -> /OUT2
- X1 pad 5: /Vin -> GND
- X1 pad 6: /OUT4 -> /OUT3
- X1 pad 7: /OUT3 -> GND
- X1 pad 8: /OUT2 -> /OUT4
- X1 pad 9: /OUT1 -> GND
Other:
- board text removed: "SWD"

Commit message: hardware update
Parts:
- added U10: LTV-354T, SOIC_Packages:SO-4_4.4x3.6mm_Pitch2.54mm, F.Cu at (87.2, 51.8)
- added U9: LTV-354T, SOIC_Packages:SO-4_4.4x3.6mm_Pitch2.54mm, F.Cu at (80.8, 51.8)
- U5, U8: value MOCD207M -> LTV-354T; footprint Housings_SOIC:SOIC-8_3.9x4.9mm_Pitch1.27mm -> SOIC_Packages:SO-4_4.4x3.6mm_Pitch2.54mm
- moved R19 10.9 mm to (97.9, 56.8)
- moved U8 10.2 mm to (71.9, 53.0), turned to 270 degrees
- moved R10 9.37 mm to (65.6, 61.3), turned to 0 degrees
- moved R21 6.35 mm to (94.8, 47.9)
- moved R8 5.12 mm to (91.6, 47.9), turned to 0 degrees
- moved R5 4.96 mm to (84.0, 51.8), turned to 90 degrees
- moved U5 3.81 mm to (66.8, 53.0), turned to 270 degrees
- moved R18 2.69 mm to (75.1, 54.9)
- moved R31 2.62 mm to (75.7, 48.6), turned to 90 degrees
- moved R4 2.29 mm to (77.6, 51.8)
- moved R17 1.80 mm to (68.1, 59.4)
- moved R30 1.42 mm to (73.2, 58.7)
- moved R20 0.90 mm to (84.0, 48.6), turned to 90 degrees
- moved R32 0.90 mm to (77.6, 48.6), turned to 90 degrees
Connections:
- U1 pad 13: Net-(U1-Pad13) -> /OPTO2
- U1 pad 14: Net-(U1-Pad14) -> /OPTO1
- U1 pad 6: Net-(U1-Pad6) -> /OPTO4
- U1 pad 7: Net-(U1-Pad7) -> /OPTO3
- U5 pad 3: Net-(R4-Pad1) -> GND
- U5 pad 4: VCOM -> /OPTO1
- U8 pad 1: Net-(R5-Pad1) -> Net-(R4-Pad1)
- U8 pad 3: Net-(R8-Pad1) -> GND
- U8 pad 4: VCOM -> /OPTO2

Commit message: libs update
Parts:
- removed D13, D14, D15: LED, LEDs:LED-0603
- removed Q5, Q7: BSS138, TO_SOT_Packages_SMD:SOT-23
- removed R33, R34, R35, R36: 470, Resistors_SMD:R_0603
- added D1: LED, LEDs:LED_0603_HandSoldering, F.Cu at (112.6, 80.2)
- added D2: TVS, Diodes_SMD:D_SMA, F.Cu at (114.2, 77.7)
- added D3: LED, LEDs:LED_0603_HandSoldering, F.Cu at (122.5, 84.6)
- added Q3: BSS138, Package_TO_SOT_SMD:SOT-23, F.Cu at (112.4, 85.7)
- added Q4: BSS138, Package_TO_SOT_SMD:SOT-23, F.Cu at (124.3, 77.7)
- added R24: 10k, Resistors_SMD:R_0603, F.Cu at (110.7, 99.7)
- added R25: 470, Resistors_SMD:R_0603, F.Cu at (110.7, 98.2)
- added R26: 10k, Resistors_SMD:R_0603, F.Cu at (119.0, 98.2)
- added R27: 470, Resistors_SMD:R_0603, F.Cu at (119.0, 99.7)
- D10, D4, D5, D7, D8: footprint Diodes_SMD:SMA_Standard -> Diodes_SMD:D_SMA
- D11, D9: value TVS -> LED; footprint Diodes_SMD:SMA_Standard -> LEDs:LED_0603_HandSoldering
- D12: value LED -> TVS; footprint LEDs:LED-0603 -> Diodes_SMD:D_SMA
- Q1, Q2: footprint TO_SOT_Packages_SMD:SOT-23 -> Package_TO_SOT_SMD:SOT-23
- R2, R7: value 10k -> 470
Connections:
- D10 pad 1: /OUT2 -> GND
- D10 pad 2: GND -> /OUT3
- D11 pad 1: /OUT1 -> Net-(D11-Pad1)
- D11 pad 2: GND -> +3V3
- D12 pad 1: Net-(D12-Pad1) -> GND
- D12 pad 2: +3V3 -> /OUT4
- D8 pad 1: /OUT4 -> GND
- D8 pad 2: GND -> /OUT2
- D9 pad 1: /OUT3 -> Net-(D9-Pad1)
- D9 pad 2: GND -> +3V3
- R2 pad 1: Net-(R2-Pad1) -> Net-(Q1-Pad3)
- R2 pad 2: +3V3 -> Net-(D1-Pad1)
- R7 pad 1: Net-(R7-Pad1) -> Net-(Q2-Pad3)
- R7 pad 2: +3V3 -> Net-(D3-Pad1)
- U2 pad 4: /Vin -> /dig_output/Vin
- U3 pad 1: Net-(R2-Pad1) -> Net-(R6-Pad1)
- U3 pad 4: /Vin -> /dig_output/Vin
- U6 pad 1: Net-(R6-Pad1) -> Net-(R24-Pad1)
- U6 pad 4: /Vin -> /dig_output/Vin
- U7 pad 1: Net-(R7-Pad1) -> Net-(R26-Pad1)
- U7 pad 4: /Vin -> /dig_output/Vin
