File: hardware/esp32control/esp32control.kicad_pcb (KiCad board)
At the start: 2 copper layers, 67.6 x 85.9 mm, 87 parts, among them J1 Conn_02x10_Odd_Even, Q1 BSS138, Q2 BSS138, Q3 BSS138, Q4 BSS138, Q5 BSS138, Q6 BSS138, Q7 MMBT3904, Q8 MMBT3904, SW1 Boot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

Commit message: bom update
Parts:
- removed REF**: OSHW-Logo2_7.3x6mm_SilkScreen, Symbol:OSHW-Logo2_7.3x6mm_SilkScreen
- C28: value CP_Small -> 100u 50V
- D10, D12, D2, D7, D8: value TVS -> SMAJ26CAQ
- D13, D6: value D_Zener_Small -> SMAZ7V5
- R14, R15: value tbd -> 100

Commit message: kicad6 update
Other:
- net class Default removed
