File: hardware/revc/esp32control.kicad_pcb (KiCad board)
At the start: 2 copper layers, 67.6 x 85.9 mm, 96 parts, among them J1 Conn_02x10_Odd_Even, Q101 2N7002, Q102 2N7002, Q202 DMP4015SK3, Q302 DMP4015SK3, Q402 DMP4015SK3, Q502 DMP4015SK3, Q7 MMBT3904, Q8 MMBT3904, SW1 Boot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

Commit message: fixed erc
Connections:
- net /OPTO3 renamed /IO35
- net /OPTO4 renamed /IO34
- net /dig_output/Out renamed /OUT1
- U1 pad 26: /IO4 -> unconnected-(U1-IO4-Pad26)
- U1 pad 37: /IO23 -> unconnected-(U1-IO23-Pad37)
