File: hardware/revc/esp32control.kicad_pcb (KiCad board)
At the start: 2 copper layers, 67.6 x 85.9 mm, 96 parts, among them J1 Conn_02x10_Odd_Even, Q101 2N7002, Q102 2N7002, Q202 DMP4015SK3, Q302 DMP4015SK3, Q402 DMP4015SK3, Q502 DMP4015SK3, Q7 MMBT3904, Q8 MMBT3904, SW1 Boot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

Commit message: updated wroom32 fp
Parts:
- U1: footprint ESP32-footprints-Lib:ESP32-WROOM -> RF_Module:ESP32-WROOM-32U
- moved U1 3.25 mm to (102.9, 76.6), turned to -90 degrees
Routing:
- net GND: track 184.7 -> 171.4 mm
