File: hardware/revc/esp32control.kicad_sch (KiCad schematic)
At the start: 60 parts, among them J1 Conn_02x10_Odd_Even, Q101 2N7002, Q102 2N7002, Q7 MMBT3904, Q8 MMBT3904, SW1 Boot, SW2 Reset, U1 ESP32-WROOM, U10 EL3H7, U101 TPS5430DDA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

Commit message: fixed erc
Connections:
- net dig_output/Out is gone; now on net OUT1: U11.2
- net IO23: no longer names the net of U1.37 (IO23)
- net IO4: no longer names the net of U1.26 (IO4)
- net OPTO3 renamed IO35
- net OPTO4 renamed IO34
- no-connect marks 13 -> 15
Changed lines of the file:
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@@
   (junction (at 280.67 30.48) (diameter 0) (color 0 0 0 0)
   )
+  (no_connect (at 160.02 119.38))
   (no_connect (at 160.02 139.7))
   (no_connect (at 113.03 151.13))
   (no_connect (at 113.03 153.67))
+  (no_connect (at 226.06 35.56))
   (no_connect (at 138.43 165.1))
   (no_connect (at 133.35 165.1))
   (no_connect (at 135.89 165.1))
   (no_connect (at 146.05 165.1))
-  (no_connect (at 224.79 30.48))
   (no_connect (at 148.59 165.1))
   (no_connect (at 143.51 165.1))
@@
   (no_connect (at 130.81 165.1))
   (no_connect (at 140.97 165.1))
+  (no_connect (at 160.02 147.32))
   (wire (pts (xy 226.06 25.4) (xy 219.71 25.4))
     (stroke (width 0) (type default))
@@
     (stroke (width 0) (type default))
   )
-  (wire (pts (xy 224.79 30.48) (xy 226.06 30.48))
-    (stroke (width 0) (type default))
-  )
   (wire (pts (xy 280.67 38.1) (xy 280.67 39.37))
     (stroke (width 0) (type default))
@@
     (stroke (width 0) (type default))
   )
-  (wire (pts (xy 211.455 19.685) (xy 212.09 19.685))
-    (stroke (width 0) (type default))
-  )
   (wire (pts (xy 106.68 48.26) (xy 104.14 48.26))
     (stroke (width 0) (type default))
@@
     (stroke (width 0) (type default))
   )
-  (wire (pts (xy 160.02 147.32) (xy 168.91 147.32))
-    (stroke (width 0) (type default))
-  )
-  (wire (pts (xy 160.02 119.38) (xy 168.91 119.38))
-    (stroke (width 0) (type default))
-  )
   (wire (pts (xy 163.83 40.64) (xy 173.99 40.64))
     (stroke (width 0) (type default))
@@
     (effects (font (size 1.524 1.524)) (justify left bottom))
   )
-  (label "OPTO3" (at 62.23 163.83 0) (fields_autoplaced)
+  (label "IO35" (at 101.6 135.89 0) (fields_autoplaced)
     (effects (font (size 1.524 1.524)) (justify left bottom))
   )
@@
     (effects (font (size 1.524 1.524)) (justify left bottom))
   )
-  (label "OPTO4" (at 62.23 180.34 0) (fields_autoplaced)
+  (label "IO34" (at 101.6 133.35 0) (fields_autoplaced)
     (effects (font (size 1.524 1.524)) (justify left bottom))
   )
@@
     (effects (font (size 1.524 1.524)) (justify left bottom))
   )
-  (label "OPTO2" (at 62.23 139.7 0) (fields_autoplaced)
-    (effects (font (size 1.524 1.524)) (justify left bottom))
-  )
-  (label "IO23" (at 162.56 119.38 0) (fields_autoplaced)
-    (effects (font (size 1.27 1.27)) (justify left bottom))
-  )
   (label "CH4" (at 18.415 71.755 180) (fields_autoplaced)
     (effects (font (size 1.524 1.524)) (justify right bottom))
@@
     (effects (font (size 1.524 1.524)) (justify right bottom))
   )
-  (label "OUT1" (at 51.3955 25.4025 180) (fields_autoplaced)
+  (label "OUT1" (at 51.435 25.4 180) (fields_autoplaced)
     (effects (font (size 1.524 1.524)) (justify right bottom))
   )
@@
     (effects (font (size 1.27 1.27)) (justify left bottom))
   )
-  (label "OPTO1" (at 62.23 123.19 0) (fields_autoplaced)
-    (effects (font (size 1.524 1.524)) (justify left bottom))
-  )
   (label "+5V" (at 227.33 66.04 0) (fields_autoplaced)
     (effects (font (size 1.524 1.524)) (justify left bottom))
@@
     (effects (font (size 1.27 1.27)) (justify left bottom))
   )
-  (label "IO4" (at 162.56 147.32 0) (fields_autoplaced)
-    (effects (font (size 1.524 1.524)) (justify left bottom))
-  )
   (label "RTS" (at 167.64 27.94 0) (fields_autoplaced)
     (effects (font (size 1.27 1.27)) (justify left bottom))
@@
       (effects (font (size 0.762 0.762)) hide)
     )
-    (property "Datasheet" "" (at 186.69 154.94 0)
+    (property "Datasheet" "~" (at 186.69 154.94 0)
       (effects (font (size 0.762 0.762)))
     )
@@
       (effects (font (size 0.762 0.762)) hide)
     )
-    (property "Datasheet" "" (at 200.66 144.78 0)
+    (property "Datasheet" "~" (at 200.66 144.78 0)
       (effects (font (size 0.762 0.762)))
     )
@@
       (effects (font (size 0.762 0.762)) hide)
     )
-    (property "Datasheet" "" (at 59.69 119.38 0)
+    (property "Datasheet" "~" (at 59.69 119.38 0)
       (effects (font (size 0.762 0.762)))
     )
@@
       (effects (font (size 0.762 0.762)) hide)
     )
-    (property "Datasheet" "" (at 59.69 135.89 0)
+    (property "Datasheet" "~" (at 59.69 135.89 0)
       (effects (font (size 0.762 0.762)))
     )
@@
       (effects (font (size 0.762 0.762)) hide)
     )
-    (property "Datasheet" "" (at 185.42 128.27 0)
+    (property "Datasheet" "~" (at 185.42 128.27 0)
       (effects (font (size 0.762 0.762)))
     )
@@
       (effects (font (size 0.762 0.762)) hide)
     )
-    (property "Datasheet" "" (at 199.39 118.11 0)
+    (property "Datasheet" "~" (at 199.39 118.11 0)
       (effects (font (size 0.762 0.762)))
     )
@@
       (effects (font (size 0.762 0.762)) hide)
     )
-    (property "Datasheet" "" (at 105.41 125.73 0)
+    (property "Datasheet" "~" (at 105.41 125.73 0)
       (effects (font (size 0.762 0.762)))
     )
@@
       (effects (font (size 0.762 0.762)) hide)
     )
-    (property "Datasheet" "" (at 59.69 160.02 0)
+    (property "Datasheet" "~" (at 59.69 160.02 0)
       (effects (font (size 0.762 0.762)))
     )
@@
       (effects (font (size 0.762 0.762)) hide)
     )
-    (property "Datasheet" "" (at 59.69 176.53 0)
+    (property "Datasheet" "~" (at 59.69 176.53 0)
       (effects (font (size 0.762 0.762)))
     )
@@
       (effects (font (size 0.762 0.762)) hide)
     )
-    (property "Datasheet" "" (at 35.56 123.19 0)
+    (property "Datasheet" "~" (at 35.56 123.19 0)
       (effects (font (size 0.762 0.762)))
     )
@@
       (effects (font (size 0.762 0.762)) hide)
     )
-    (property "Datasheet" "" (at 35.56 139.7 0)
+    (property "Datasheet" "~" (at 35.56 139.7 0)
       (effects (font (size 0.762 0.762)))
     )
@@
       (effects (font (size 0.762 0.762)) hide)
     )
-    (property "Datasheet" "" (at 35.56 163.83 0)
+    (property "Datasheet" "~" (at 35.56 163.83 0)
       (effects (font (size 0.762 0.762)))
     )
@@
       (effects (font (size 0.762 0.762)) hide)
     )
-    (property "Datasheet" "" (at 35.56 180.34 0)
+    (property "Datasheet" "~" (at 35.56 180.34 0)
       (effects (font (size 0.762 0.762)))
     )
@@
       (effects (font (size 0.762 0.762)) hide)
     )
-    (property "Datasheet" "" (at 193.04 69.85 0)
+    (property "Datasheet" "~" (at 193.04 69.85 0)
       (effects (font (size 0.762 0.762)))
     )
@@
       (effects (font (size 0.762 0.762)) hide)
     )
-    (property "Datasheet" "" (at 187.96 69.85 0)
+    (property "Datasheet" "~" (at 187.96 69.85 0)
       (effects (font (size 0.762 0.762)))
     )
@@
       (effects (font (size 0.762 0.762)) hide)
     )
-    (property "Datasheet" "" (at 222.25 69.85 0)
+    (property "Datasheet" "~" (at 222.25 69.85 0)
       (effects (font (size 0.762 0.762)))
     )
@@
       (effects (font (size 0.762 0.762)) hide)
     )
-    (property "Datasheet" "" (at 227.33 69.85 0)
+    (property "Datasheet" "~" (at 227.33 69.85 0)
       (effects (font (size 0.762 0.762)))
     )
@@
       (effects (font (size 0.762 0.762)) hide)
     )
-    (property "Datasheet" "" (at 252.095 71.12 0)
+    (property "Datasheet" "~" (at 252.095 71.12 0)
       (effects (font (size 0.762 0.762)))
     )
@@
       (effects (font (size 0.762 0.762)) hide)
     )
-    (property "Datasheet" "" (at 110.49 48.26 0)
+    (property "Datasheet" "~" (at 110.49 48.26 0)
       (effects (font (size 0.762 0.762)))
     )
@@
       (effects (font (size 0.762 0.762)) hide)
     )
-    (property "Datasheet" "" (at 110.49 45.72 0)
+    (property "Datasheet" "~" (at 110.49 45.72 0)
       (effects (font (size 0.762 0.762)))
     )
@@
       (effects (font (size 1.27 1.27) italic) (justify left) hide)
     )
-    (property "Datasheet" "https://www.fairchildsemi.com/datasheets/2N/2N3904.pdf" (at 232.41 129.54 0)
+    (property "Datasheet" "https://www.onsemi.com/pdf/datasheet/pzt3904-d.pdf" (at 232.41 129.54 0)
       (effects (font (size 1.27 1.27)) (justify left) hide)
     )
@@
       (effects (font (size 1.27 1.27) italic) (justify left) hide)
     )
-    (property "Datasheet" "https://www.fairchildsemi.com/datasheets/2N/2N3904.pdf" (at 232.41 144.78 0)
+    (property "Datasheet" "https://www.onsemi.com/pdf/datasheet/pzt3904-d.pdf" (at 232.41 144.78 0)
       (effects (font (size 1.27 1.27)) (justify left) hide)
     )
@@
       (effects (font (size 0.762 0.762)) hide)
     )
-    (property "Datasheet" "" (at 246.38 129.54 0)
+    (property "Datasheet" "~" (at 246.38 129.54 0)
       (effects (font (size 0.762 0.762)))
     )
@@
       (effects (font (size 0.762 0.762)) hide)
     )
-    (property "Datasheet" "" (at 246.38 144.78 0)
+    (property "Datasheet" "~" (at 246.38 144.78 0)
       (effects (font (size 0.762 0.762)))
     )
@@
       (effects (font (size 0.762 0.762)) hide)
     )
-    (property "Datasheet" "" (at 132.715 31.75 0)
+    (property "Datasheet" "~" (at 132.715 31.75 0)
       (effects (font (size 0.762 0.762)))
     )
@@
       (effects (font (size 0.762 0.762)) hide)
     )
-    (property "Datasheet" "" (at 181.61 31.75 0)
+    (property "Datasheet" "~" (at 181.61 31.75 0)
       (effects (font (size 0.762 0.762)))
     )

Commit message: updated wroom32 fp
Parts:
- U1: footprint ESP32-footprints-Lib:ESP32-WROOM -> RF_Module:ESP32-WROOM-32U
Changed lines of the file:
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@@
       (effects (font (size 1.524 1.524)))
     )
-    (property "Footprint" "ESP32-footprints-Lib:ESP32-WROOM" (at 146.05 104.14 0)
+    (property "Footprint" "RF_Module:ESP32-WROOM-32U" (at 146.05 104.14 0)
       (effects (font (size 1.524 1.524)) hide)
     )

Commit message: updated sch, pcb, bom
Parts:
- removed R19: nb, Resistor_SMD:R_0603_1608Metric, symbol Device:R
- C2: JLCPCB# (none) -> C57112
- C23: value 100n 50V -> 1u 25V; JLCPCB# C14663 -> C15849; Mouser 80-C0603C104M5R -> (none)
- R101: value 10k -> 12k; JLCPCB# C25804 -> C22790
- R102: value 3k24 -> 3k9; JLCPCB# (none) -> C23018
- R11, R14, R15, R23: JLCPCB# (none) -> C22775
- R3, R4, R5, R8: JLCPCB# (none) -> C22843
- SW1: footprint switches:SMD_Switch_6.5x6 -> Button_Switch_SMD:SW_SPST_TL3342; symbol standard:Switch_4P -> Switch:SW_Push; JLCPCB# (none) -> C318884; Mouser 667-EVQ-Q2B03W -> (none)
- SW2: footprint switches:SMD_Switch_6.5x6 -> Button_Switch_SMD:SW_SPST_TL3342; symbol standard:Switch_4P -> Switch:SW_Push; JLCPCB# (none) -> C318884
- U1: footprint RF_Module:ESP32-WROOM-32U -> RF_Module:ESP32-WROOM-32UE; JLCPCB# (none) -> C3013937
Connections:
- net nBoot: now also SW1.2; no longer SW1.B, SW1.B'
- net nReset: now also SW2.2; no longer SW2.B, SW2.B'
- new net: R11.1, SW2.1
- new net: R23.1, SW1.1
