File: hardware/revc/esp32control.kicad_sch (KiCad schematic)
At the start: 60 parts, among them J1 Conn_02x10_Odd_Even, Q101 2N7002, Q102 2N7002, Q7 MMBT3904, Q8 MMBT3904, SW1 Boot, SW2 Reset, U1 ESP32-WROOM, U10 EL3H7, U101 TPS5430DDA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

Commit message: workflow fix (#2)
* remove inner layer in yaml

* fixed erc

* fixed drc

* updated wroom32 fp

* updated kibot

* updated pcb

* updated pcb

* updated yml

* yml updates

* fixed layer entries

* updated sch, pcb, bom

* reduced drc verbosity
Parts:
- removed R19: nb, Resistor_SMD:R_0603_1608Metric, symbol Device:R
- C2: JLCPCB# (none) -> C57112
- C23: value 100n 50V -> 1u 25V; JLCPCB# C14663 -> C15849; Mouser 80-C0603C104M5R -> (none)
- R101: value 10k -> 12k; JLCPCB# C25804 -> C22790
- R102: value 3k24 -> 3k9; JLCPCB# (none) -> C23018
- R11, R14, R15, R23: JLCPCB# (none) -> C22775
- R3, R4, R5, R8: JLCPCB# (none) -> C22843
- SW1: footprint switches:SMD_Switch_6.5x6 -> Button_Switch_SMD:SW_SPST_TL3342; symbol standard:Switch_4P -> Switch:SW_Push; JLCPCB# (none) -> C318884; Mouser 667-EVQ-Q2B03W -> (none)
- SW2: footprint switches:SMD_Switch_6.5x6 -> Button_Switch_SMD:SW_SPST_TL3342; symbol standard:Switch_4P -> Switch:SW_Push; JLCPCB# (none) -> C318884
- U1: footprint ESP32-footprints-Lib:ESP32-WROOM -> RF_Module:ESP32-WROOM-32UE; JLCPCB# (none) -> C3013937
Connections:
- net dig_output/Out is gone; now on net OUT1: U11.2
- net nBoot: now also SW1.2; no longer SW1.B, SW1.B'
- net nReset: now also SW2.2; no longer SW2.B, SW2.B'
- net IO23: no longer names the net of U1.37 (IO23)
- net IO4: no longer names the net of U1.26 (IO4)
- net OPTO3 renamed IO35
- net OPTO4 renamed IO34
- new net: R11.1, SW2.1
- new net: R23.1, SW1.1
- no-connect marks 13 -> 15
