File: hardware/revc/dig_output.kicad_sch (KiCad schematic)
At the start: 9 parts, among them Q202 DMP4015SK3, U5 EL3H7

Commit message: workflow fix (#2)
* remove inner layer in yaml

* fixed erc

* fixed drc

* updated wroom32 fp

* updated kibot

* updated pcb

* updated pcb

* updated yml

* yml updates

* fixed layer entries

* updated sch, pcb, bom

* reduced drc verbosity
Parts:
- D201: value BZX84Cxx -> BZX84C10; JLCPCB# (none) -> C118575
- Q202: value DMP4015SK3 -> HSU4113; JLCPCB# C461089 -> C701017; LCSC# C513222 -> (none)
Changed lines of the file:
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@@
       (effects (font (size 1.27 1.27)) (justify left))
     )
-    (property "Value" "DMP4015SK3" (at 150.495 73.66 0)
+    (property "Value" "HSU4113" (at 150.495 73.66 0)
       (effects (font (size 1.27 1.27)) (justify left))
     )
@@
       (effects (font (size 1.27 1.27)) hide)
     )
-    (property "LCSC#" "C513222" (at 145.415 74.93 0)
+    (property "LCSC#" "" (at 145.415 74.93 0)
       (effects (font (size 1.27 1.27)) hide)
     )
-    (property "JLCPCB#" "C461089" (at 145.415 74.93 0)
+    (property "JLCPCB#" "C701017" (at 145.415 74.93 0)
       (effects (font (size 1.27 1.27)) hide)
     )
@@
       (effects (font (size 1.27 1.27)))
     )
-    (property "Value" "BZX84Cxx" (at 136.525 67.31 0)
+    (property "Value" "BZX84C10" (at 136.525 67.31 0)
       (effects (font (size 1.27 1.27)))
     )
@@
       (effects (font (size 1.27 1.27)) hide)
     )
+    (property "JLCPCB#" "C118575" (at 140.335 67.31 0)
+      (effects (font (size 1.27 1.27)) hide)
+    )
